File: MicroPicoDriveCartridge/MicroPicoDriveCartridge.kicad_sch (KiCad schematic)
At the start: 10 parts, among them J1 Edge Connector, J2 0.96 IPS ST7735S, J3 K1..K4, J4 DM3D-SF, J6 Micro_SD_Card_Det_Hirose_DM3AT

Commit message: Stagger cartridge edge fingers for hot-swap mating order
GND (pin 3) and the GND-tied UI_DETECT (pin 14) keep the full 8 mm
length and mate first, +3V3 is retracted 1 mm, and all signal fingers
are retracted 1.75 mm so they mate last and break first. Gerbers and
iBOM regenerated; the Edge library footprint is synced with the board.
Parts:
- J1: footprint CartridgeComponents:Edge -> My Footprint Library:MicroPicoDrive Cartridge Edge
Changed lines of the file:
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@@
 			)
 		)
-		(property "Footprint" "CartridgeComponents:Edge"
+		(property "Footprint" "My Footprint Library:MicroPicoDrive Cartridge Edge"
 			(at 60.96 123.19 0)
 			(hide yes)
