File: MicroPicoDrive/MicroPicoDrive.kicad_sch (KiCad schematic)
At the start: 19 parts, among them IC1 SN74LVC1T45DBVR, IC2 SN74LVC1T45DBVR, IC3 TXU0304QPWRQ1, J1 Conn_02x16, J2 QL_CONN, J3 PicoBlade-53261-0371, U1 LM7805_TO220, U2 Pico, U3 LM1117MP-5.0, U4 AMS1117-5.0

Commit message: Change C7 and C8 to 0805 hand-solder footprints
The two capacitors move from C_0603_1608Metric to
C_0805_2012Metric_Pad1.18x1.45mm_HandSolder in both the schematic
and the board. Gerbers and drill files are regenerated from the
updated board, and the DRC silkscreen text height, thickness and
back-layer mirroring checks are set to ignore.
Parts:
- C7, C8: footprint Capacitor_SMD:C_0603_1608Metric -> Capacitor_SMD:C_0805_2012Metric_Pad1.18x1.45mm_HandSolder
Changed lines of the file:
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@@
 			)
 		)
-		(property "Footprint" "Capacitor_SMD:C_0603_1608Metric"
+		(property "Footprint" "Capacitor_SMD:C_0805_2012Metric_Pad1.18x1.45mm_HandSolder"
 			(at 218.1352 52.07 0)
 			(hide yes)
@@
 			)
 		)
-		(property "Footprint" "Capacitor_SMD:C_0603_1608Metric"
+		(property "Footprint" "Capacitor_SMD:C_0805_2012Metric_Pad1.18x1.45mm_HandSolder"
 			(at 195.2752 52.07 0)
 			(hide yes)
